File: Wii Guitar PCB/Wii Guitar.kicad_sch (KiCad schematic)
At the start: 35 parts, among them J1 USB_C_Receptacle_USB2.0, J2 Wii Guitar, J3 Battery, SW1 SW_Push, U1 ESP32-WROOM-32D, U2 LM66100DCKT, U3 BQ24090DGQ, U4 FT230XQ, U5 TPS63001

Commit message: Added Final Design
Parts:
- removed H1, H2, H3, H4: MountingHole, MountingHole:MountingHole_3.2mm_M3, symbol Mechanical:MountingHole
- added H1, H2, H3, H4: MountingHole_Pad, MountingHole:MountingHole_3.2mm_M3_ISO14580_Pad_TopBottom, symbol Mechanical:MountingHole_Pad
- C1, C5: value 0.1u -> 0.1uF; footprint Capacitor_SMD:C_0805_2012Metric -> Capacitor_SMD:C_0805_2012Metric_Pad1.18x1.45mm_HandSolder
- C10: value 10u -> 10uF; footprint Capacitor_SMD:C_0805_2012Metric -> Capacitor_SMD:C_0805_2012Metric_Pad1.18x1.45mm_HandSolder; Digikey 1276-6471-1-ND -> 1276-1096-1-ND
- C11: value 33u -> 33uF; footprint Capacitor_SMD:C_0805_2012Metric -> Capacitor_SMD:C_0805_2012Metric_Pad1.18x1.45mm_HandSolder; Digikey 1276-6471-1-ND -> 445-8238-1-ND
- C2: value 10n -> 10nF; footprint Capacitor_SMD:C_0805_2012Metric -> Capacitor_SMD:C_0805_2012Metric_Pad1.18x1.45mm_HandSolder
- C3, C6: value 1u -> 1uF; footprint Capacitor_SMD:C_0805_2012Metric -> Capacitor_SMD:C_0805_2012Metric_Pad1.18x1.45mm_HandSolder
- C4: value 10u -> 10uF; footprint Capacitor_SMD:C_0805_2012Metric -> Capacitor_SMD:C_0805_2012Metric_Pad1.18x1.45mm_HandSolder
- C7: value 4.7u -> 4.7uF; footprint Capacitor_SMD:C_0805_2012Metric -> Capacitor_SMD:C_0805_2012Metric_Pad1.18x1.45mm_HandSolder; Digikey 1276-6471-1-ND -> 1276-1244-1-ND
- C8, C9: value 47p -> 47pF; footprint Capacitor_SMD:C_0805_2012Metric -> Capacitor_SMD:C_0805_2012Metric_Pad1.18x1.45mm_HandSolder
- FB1: value 600 -> 600H
- J1: footprint (none) -> Connector_USB:USB_C_Receptacle_JAE_DX07S024WJ1R350; Digikey (none) -> 670-2949-1-ND
- J3: footprint (none) -> Connector_JST:JST_PH_B2B-PH-K_1x02_P2.00mm_Vertical
- L1: value 1.5u -> 1.5uH; footprint (none) -> Inductor_SMD:L_Wuerth_MAPI-1610; Digikey (none) -> 732-78438313015CT-ND
- R1: value 10k -> 10kR; footprint Resistor_SMD:R_0805_2012Metric -> Resistor_SMD:R_0805_2012Metric_Pad1.20x1.40mm_HandSolder
- R2: value 560 -> 560R; footprint Resistor_SMD:R_0805_2012Metric -> Resistor_SMD:R_0805_2012Metric_Pad1.20x1.40mm_HandSolder
- R3, R4: value 5.1k -> 5.1kR; footprint Resistor_SMD:R_0805_2012Metric -> Resistor_SMD:R_0805_2012Metric_Pad1.20x1.40mm_HandSolder; Digikey 738-RMCF0805FT27R0CT-ND -> P5.1KDACT-ND
- R5: value 1k -> 1kR; footprint Resistor_SMD:R_0805_2012Metric -> Resistor_SMD:R_0805_2012Metric_Pad1.20x1.40mm_HandSolder; Digikey 738-RMCF0805FT27R0CT-ND -> P1.0KBFCT-ND
- R6: value 2k -> 2kR; footprint Resistor_SMD:R_0805_2012Metric -> Resistor_SMD:R_0805_2012Metric_Pad1.20x1.40mm_HandSolder; Digikey 738-RMCF0805FT27R0CT-ND -> P2.0KBSCT-ND
- R7, R8: value 27 -> 27R; footprint Resistor_SMD:R_0805_2012Metric -> Resistor_SMD:R_0805_2012Metric_Pad1.20x1.40mm_HandSolder
- R9: value 10k -> 10kR; footprint Resistor_SMD:R_0805_2012Metric -> Resistor_SMD:R_0805_2012Metric_Pad1.20x1.40mm_HandSolder; Digikey 738-RMCF0805FT27R0CT-ND -> RNCP0805FTD10K0CT-ND
- U2: footprint SOT65P210X110-6N -> Package_TO_SOT_SMD:SOT-363_SC-70-6
Connections:
- net GND: now also H1.1, H2.1, H3.1, H4.1
